File: schematics/draw.kicad_pcb (KiCad board)
At the start: 2 copper layers, 50 x 40 mm, 37 parts, among them P1 I2C, P2 UART, P3 DBG, P4 USB_OTG, P5 Power_IN, P6 Power_OUT, SW1 SW_Push, U1 EFM32HG309, U2 TPD4E002, U3 INA260

Commit message: added logo and url silkscreen
Parts:
- added REF***: OSHW-Logo_5.7x6mm_SilkScreen, Symbols:OSHW-Logo_5.7x6mm_SilkScreen, B.Cu at (64.3, 112.6)
Other:
- board text added: "chinmay.audio/draw"
- board text added: "draw v1.0 7/2/2017"
