File: schematics/measure.sch (KiCad schematic (older format))
At the start: 12 parts, among them P5 Power_IN, P6 Power_OUT, U3 INA260

Commit message: first layout
Connections:
- net I2C_SDA: no longer R14.1, R15.1
- net at C5.1, U3.1 (IN+), U3.12 (VBUS)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: now also P5.1 (P1); no longer P5.2 (P2)
- net at U3.14 (IN-), U3.15 (IN-), U3.16 (IN-): now also P6.2 (P2); no longer P6.1 (P1)
- net +3V3 renamed +3.3VA
- net +3.3VA: now also R14.1, R15.1
- net GND renamed GNDA
- net GNDA: now also P5.2 (P2), P6.1 (P1); no longer P5.1 (P1), P6.2 (P2)
Other:
- moved on the sheet: P6
Changed lines of the file:
@@
 $EndComp
-$Comp
-L GND #PWR014
-U 1 1 5881C8A1
-P 4700 3750
-F 0 "#PWR014" H 4700 3500 50  0001 C CNN
-F 1 "GND" H 4700 3600 50  0000 C CNN
-F 2 "" H 4700 3750 50  0000 C CNN
-F 3 "" H 4700 3750 50  0000 C CNN
-	1    4700 3750
-	1    0    0    -1
-$EndComp
-$Comp
-L +3.3V #PWR015
-U 1 1 5881C8BE
-P 4700 3650
-F 0 "#PWR015" H 4700 3500 50  0001 C CNN
-F 1 "+3.3V" H 4700 3790 50  0000 C CNN
-F 2 "" H 4700 3650 50  0000 C CNN
-F 3 "" H 4700 3650 50  0000 C CNN
-	1    4700 3650
-	1    0    0    -1
-$EndComp
-Wire Wire Line
-	4700 3650 4850 3650
-Wire Wire Line
-	4700 3750 4850 3750
 $Comp
 L R_Small R11
@@
 	0    1    1    0
 $EndComp
-Wire Wire Line
-	5150 4150 5050 4150
-Wire Wire Line
-	5150 4250 5050 4250
-$Comp
-L GND #PWR016
-U 1 1 5881C9D1
-P 4700 4250
-F 0 "#PWR016" H 4700 4000 50  0001 C CNN
-F 1 "GND" H 4700 4100 50  0000 C CNN
-F 2 "" H 4700 4250 50  0000 C CNN
-F 3 "" H 4700 4250 50  0000 C CNN
-	1    4700 4250
-	1    0    0    -1
-$EndComp
-$Comp
-L +3.3V #PWR017
-U 1 1 5881C9D7
-P 4700 4150
-F 0 "#PWR017" H 4700 4000 50  0001 C CNN
-F 1 "+3.3V" H 4700 4290 50  0000 C CNN
-F 2 "" H 4700 4150 50  0000 C CNN
-F 3 "" H 4700 4150 50  0000 C CNN
-	1    4700 4150
-	1    0    0    -1
-$EndComp
-Wire Wire Line
-	4700 4150 4850 4150
-Wire Wire Line
-	4700 4250 4850 4250
-Wire Wire Line
-	5050 3650 5050 3800
-Wire Wire Line
-	5150 3950 5150 4250
-Wire Wire Line
-	6700 4000 6700 4100
-$Comp
-L GND #PWR018
-U 1 1 5881CC9E
-P 6700 4100
-F 0 "#PWR018" H 6700 3850 50  0001 C CNN
-F 1 "GND" H 6700 3950 50  0000 C CNN
-F 2 "" H 6700 4100 50  0000 C CNN
-F 3 "" H 6700 4100 50  0000 C CNN
-	1    6700 4100
-	1    0    0    -1
-$EndComp
 Text HLabel 7150 4000 2    60   Input ~ 0
 GND
 Text HLabel 7150 3900 2    60   Input ~ 0
 3.3V
-Wire Wire Line
-	6700 4000 7150 4000
-Wire Wire Line
-	6700 3900 7150 3900
-$Comp
-L +3.3V #PWR019
-U 1 1 5881CD56
-P 6950 3850
-F 0 "#PWR019" H 6950 3700 50  0001 C CNN
-F 1 "+3.3V" H 7050 3850 50  0000 C CNN
-F 2 "" H 6950 3850 50  0000 C CNN
-F 3 "" H 6950 3850 50  0000 C CNN
-	1    6950 3850
-	1    0    0    -1
-$EndComp
-Connection ~ 6950 3900
 $Comp
 L CONN_01X02 P6
 U 1 1 5881CF01
-P 7000 3250
-F 0 "P6" H 7000 3400 50  0000 C CNN
-F 1 "Power_OUT" V 7100 3250 50  0000 C CNN
-F 2 "Terminal_Blocks:TerminalBlock_Pheonix_MKDS1.5-2pol" H 7000 3250 50  0001 C CNN
-F 3 "" H 7000 3250 50  0000 C CNN
-	1    7000 3250
+P 7000 3100
+F 0 "P6" H 7000 3250 50  0000 C CNN
+F 1 "Power_OUT" V 7100 3100 50  0000 C CNN
+F 2 "Terminal_Blocks:TerminalBlock_Pheonix_MKDS1.5-2pol" H 7000 3100 50  0001 C CNN
+F 3 "" H 7000 3100 50  0000 C CNN
+	1    7000 3100
 	1    0    0    -1
 $EndComp
@@
 	-1   0    0    1
 $EndComp
-Wire Wire Line
-	6700 3200 6700 3400
-Connection ~ 6700 3300
-Wire Wire Line
-	6700 3200 6800 3200
-$Comp
-L GND #PWR020
-U 1 1 5881D061
-P 6800 3300
-F 0 "#PWR020" H 6800 3050 50  0001 C CNN
-F 1 "GND" H 6800 3150 50  0000 C CNN
-F 2 "" H 6800 3300 50  0000 C CNN
-F 3 "" H 6800 3300 50  0000 C CNN
-	1    6800 3300
-	1    0    0    -1
-$EndComp
-Wire Wire Line
-	5350 3100 5350 3600
-Connection ~ 5350 3300
-Wire Wire Line
-	5350 3100 4900 3100
-$Comp
-L GND #PWR021
-U 1 1 5881D145
-P 4900 3200
-F 0 "#PWR021" H 4900 2950 50  0001 C CNN
-F 1 "GND" H 4900 3050 50  0000 C CNN
-F 2 "" H 4900 3200 50  0000 C CNN
-F 3 "" H 4900 3200 50  0000 C CNN
-	1    4900 3200
-	1    0    0    -1
-$EndComp
-Connection ~ 5350 3400
 Text HLabel 7650 3550 2    60   Input ~ 0
 I2C_SDA
@@
 Text HLabel 7750 3750 2    60   Input ~ 0
 ALERT
-Wire Wire Line
-	6700 3750 7750 3750
-Wire Wire Line
-	6950 3850 6950 3900
-Connection ~ 5350 3200
-Connection ~ 6700 3400
-Connection ~ 6700 3200
 $Comp
 L R_Small R13
@@
 	1    0    0    -1
 $EndComp
-Wire Wire Line
-	7250 3200 7250 3550
-Wire Wire Line
-	7250 3200 7600 3200
-$Comp
-L +3.3V #PWR022
-U 1 1 58841F37
-P 7250 3000
-F 0 "#PWR022" H 7250 2850 50  0001 C CNN
-F 1 "+3.3V" H 7250 3140 50  0000 C CNN
-F 2 "" H 7250 3000 50  0000 C CNN
-F 3 "" H 7250 3000 50  0000 C CNN
-	1    7250 3000
-	1    0    0    -1
-$EndComp
-Wire Wire Line
-	7600 3500 7600 3750
-Connection ~ 7600 3750
-Wire Wire Line
-	6700 3650 7700 3650
-Wire Wire Line
-	6700 3550 7650 3550
-Wire Wire Line
-	7400 3400 7400 3650
-Connection ~ 7400 3650
-Connection ~ 7250 3550
-Wire Wire Line
-	7600 3200 7600 3300
-Connection ~ 7400 3200
 $Comp
 L C_Small C4
@@
 	1    0    0    -1
 $EndComp
-Wire Wire Line
-	6700 4100 6850 4100
-Connection ~ 6850 3900
 $Comp
 L C_Small C5
@@
 P 5250 3550
 F 0 "C5" H 5150 3650 50  0000 L CNN
-F 1 "1uF" H 5100 3400 50  0000 L CNN
+F 1 "1uF" H 5050 3550 50  0000 L CNN
 F 2 "Capacitors_SMD:C_0805_HandSoldering" H 5250 3550 50  0001 C CNN
 F 3 "" H 5250 3550 50  0000 C CNN
@@
 	1    0    0    -1
 $EndComp
-Wire Wire Line
-	5250 3450 5350 3450
-Connection ~ 5350 3450
-$Comp
-L GND #PWR023
-U 1 1 58847CCB
+$Comp
+L +3.3VA #PWR014
+U 1 1 588F0CB3
+P 6950 3850
+F 0 "#PWR014" H 6950 3700 50  0001 C CNN
+F 1 "+3.3VA" H 6950 3990 50  0000 C CNN
+F 2 "" H 6950 3850 50  0000 C CNN
+F 3 "" H 6950 3850 50  0000 C CNN
+	1    6950 3850
+	1    0    0    -1
+$EndComp
+$Comp
+L +3.3VA #PWR015
+U 1 1 588F18A1
+P 4700 3650
+F 0 "#PWR015" H 4700 3500 50  0001 C CNN
+F 1 "+3.3VA" H 4700 3790 50  0000 C CNN
+F 2 "" H 4700 3650 50  0000 C CNN
+F 3 "" H 4700 3650 50  0000 C CNN
+	1    4700 3650
+	1    0    0    -1
+$EndComp
+$Comp
+L +3.3VA #PWR016
+U 1 1 588F1952
+P 4700 4150
+F 0 "#PWR016" H 4700 4000 50  0001 C CNN
+F 1 "+3.3VA" H 4700 4290 50  0000 C CNN
+F 2 "" H 4700 4150 50  0000 C CNN
+F 3 "" H 4700 4150 50  0000 C CNN
+	1    4700 4150
+	1    0    0    -1
+$EndComp
+$Comp
+L +3.3VA #PWR017
+U 1 1 588F1A71
+P 7250 3000
+F 0 "#PWR017" H 7250 2850 50  0001 C CNN
+F 1 "+3.3VA" H 7250 3140 50  0000 C CNN
+F 2 "" H 7250 3000 50  0000 C CNN
+F 3 "" H 7250 3000 50  0000 C CNN
+	1    7250 3000
+	1    0    0    -1
+$EndComp
+$Comp
+L GNDA #PWR018
+U 1 1 588F1B2E
+P 4700 4250
+F 0 "#PWR018" H 4700 4000 50  0001 C CNN
+F 1 "GNDA" H 4700 4100 50  0000 C CNN
+F 2 "" H 4700 4250 50  0000 C CNN
+F 3 "" H 4700 4250 50  0000 C CNN
+	1    4700 4250
+	1    0    0    -1
+$EndComp
+$Comp
+L GNDA #PWR019
+U 1 1 588F1B73
+P 4700 3750
+F 0 "#PWR019" H 4700 3500 50  0001 C CNN
+F 1 "GNDA" H 4700 3600 50  0000 C CNN
+F 2 "" H 4700 3750 50  0000 C CNN
+F 3 "" H 4700 3750 50  0000 C CNN
+	1    4700 3750
+	1    0    0    -1
+$EndComp
+$Comp
+L GNDA #PWR020
+U 1 1 588F1C0C
+P 5050 2850
+F 0 "#PWR020" H 5050 2600 50  0001 C CNN
+F 1 "GNDA" H 5050 2700 50  0000 C CNN
+F 2 "" H 5050 2850 50  0000 C CNN
+F 3 "" H 5050 2850 50  0000 C CNN
+	1    5050 2850
+	1    0    0    -1
+$EndComp
+$Comp
+L GNDA #PWR021
+U 1 1 588F1CBD
+P 6700 2850
+F 0 "#PWR021" H 6700 2600 50  0001 C CNN
+F 1 "GNDA" H 6700 2700 50  0000 C CNN
+F 2 "" H 6700 2850 50  0000 C CNN
+F 3 "" H 6700 2850 50  0000 C CNN
+	1    6700 2850
+	1    0    0    -1
+$EndComp
+$Comp
+L GNDA #PWR022
+U 1 1 588F1D56
+P 6700 4100
+F 0 "#PWR022" H 6700 3850 50  0001 C CNN
+F 1 "GNDA" H 6700 3950 50  0000 C CNN
+F 2 "" H 6700 4100 50  0000 C CNN
+F 3 "" H 6700 4100 50  0000 C CNN
+	1    6700 4100
+	1    0    0    -1
+$EndComp
+$Comp
+L GNDA #PWR023
+U 1 1 588F1F34
 P 5250 3650
 F 0 "#PWR023" H 5250 3400 50  0001 C CNN
-F 1 "GND" H 5350 3600 50  0000 C CNN
+F 1 "GNDA" H 5250 3500 50  0000 C CNN
 F 2 "" H 5250 3650 50  0000 C CNN
 F 3 "" H 5250 3650 50  0000 C CNN
@@
 $EndComp
 Wire Wire Line
+	4700 3650 4850 3650
+Wire Wire Line
+	4700 3750 4850 3750
+Wire Wire Line
+	5150 4150 5050 4150
+Wire Wire Line
+	5150 4250 5050 4250
+Wire Wire Line
+	4700 4150 4850 4150
+Wire Wire Line
+	4700 4250 4850 4250
+Wire Wire Line
+	5050 3650 5050 3800
+Wire Wire Line
+	5150 3950 5150 4250
+Wire Wire Line
+	6700 4000 6700 4100
+Wire Wire Line
+	6700 4000 7150 4000
+Wire Wire Line
+	6700 3900 7150 3900
+Connection ~ 6950 3900
+Wire Wire Line
+	6700 3150 6700 3400
+Connection ~ 6700 3300
+Connection ~ 5350 3300
+Connection ~ 5350 3400
+Wire Wire Line
+	6700 3750 7750 3750
+Wire Wire Line
+	6950 3850 6950 3900
+Connection ~ 5350 3200
+Connection ~ 6700 3400
+Connection ~ 6700 3200
+Wire Wire Line
+	7250 3200 7250 3550
+Wire Wire Line
+	7400 3200 7600 3200
+Wire Wire Line
+	7600 3500 7600 3750
+Connection ~ 7600 3750
+Wire Wire Line
+	6700 3650 7700 3650
+Wire Wire Line
+	6700 3550 7650 3550
+Wire Wire Line
+	7400 3400 7400 3650
+Connection ~ 7400 3650
+Connection ~ 7250 3550
+Wire Wire Line
+	7600 3200 7600 3300
+Wire Wire Line
+	6700 4100 6850 4100
+Connection ~ 6850 3900
+Wire Wire Line
+	5350 3450 5250 3450
+Connection ~ 5350 3450
+Wire Wire Line
 	5350 3750 5350 3800
 Wire Wire Line
@@
 	5350 3950 5150 3950
 Connection ~ 5150 4150
+Wire Wire Line
+	5350 3200 5350 3600
+Wire Wire Line
+	5350 3200 4900 3200
+Wire Wire Line
+	4900 3100 4900 2850
+Wire Wire Line
+	4900 2850 5050 2850
+Wire Wire Line
+	6800 3050 6800 2850
+Wire Wire Line
+	6800 2850 6700 2850
+Wire Wire Line
+	6800 3150 6700 3150
+Wire Wire Line
+	7250 3000 7400 3000
+Wire Wire Line
+	7400 3000 7400 3200
+Connection ~ 7250 3000
 $EndSCHEMATC

Commit message: updated to work in kicad 5.1
Parts:
- C4, C5: symbol C_Small -> Device:C_Small
- P5, P6: symbol CONN_01X02 -> Connector:Screw_Terminal_01x02
- R10, R11, R12, R13, R14, R15, R9: symbol R_Small -> Device:R_Small
- U3: symbol INA260 -> draw:INA260
Changed lines of the file:
@@
-EESchema Schematic File Version 2
-LIBS:power
-LIBS:device
-LIBS:transistors
-LIBS:conn
-LIBS:linear
-LIBS:regul
-LIBS:74xx
-LIBS:cmos4000
-LIBS:adc-dac
-LIBS:memory
-LIBS:xilinx
-LIBS:microcontrollers
-LIBS:dsp
-LIBS:microchip
-LIBS:analog_switches
-LIBS:motorola
-LIBS:texas
-LIBS:intel
-LIBS:audio
-LIBS:interface
-LIBS:digital-audio
-LIBS:philips
-LIBS:display
-LIBS:cypress
-LIBS:siliconi
-LIBS:opto
-LIBS:atmel
-LIBS:contrib
-LIBS:valves
-LIBS:draw
-LIBS:switches
-LIBS:silabs
+EESchema Schematic File Version 4
 LIBS:draw-cache
-EELAYER 25 0
+EELAYER 29 0
 EELAYER END
 $Descr A4 11693 8268
@@
 $EndDescr
 $Comp
-L INA260 U3
+L draw:INA260 U3
 U 1 1 5881C68E
 P 5550 4200
@@
 $EndComp
 $Comp
-L R_Small R9
+L Device:R_Small R9
 U 1 1 5881C6C5
 P 4950 3650
@@
 $EndComp
 $Comp
-L R_Small R10
+L Device:R_Small R10
 U 1 1 5881C6FE
 P 4950 3750
@@
 $EndComp
 $Comp
-L R_Small R11
+L Device:R_Small R11
 U 1 1 5881C9C3
 P 4950 4150
@@
 $EndComp
 $Comp
-L R_Small R12
+L Device:R_Small R12
 U 1 1 5881C9C9
 P 4950 4250
@@
 3.3V
 $Comp
-L CONN_01X02 P6
+L Connector:Screw_Terminal_01x02 P6
 U 1 1 5881CF01
-P 7000 3100
-F 0 "P6" H 7000 3250 50  0000 C CNN
-F 1 "Power_OUT" V 7100 3100 50  0000 C CNN
-F 2 "Terminal_Blocks:TerminalBlock_Pheonix_MKDS1.5-2pol" H 7000 3100 50  0001 C CNN
-F 3 "" H 7000 3100 50  0000 C CNN
-	1    7000 3100
-	1    0    0    -1
-$EndComp
-$Comp
-L CONN_01X02 P5
-U 1 1 5881CF96
-P 4700 3150
-F 0 "P5" H 4700 3300 50  0000 C CNN
-F 1 "Power_IN" V 4800 3150 50  0000 C CNN
-F 2 "Terminal_Blocks:TerminalBlock_Pheonix_MKDS1.5-2pol" H 4700 3150 50  0001 C CNN
-F 3 "" H 4700 3150 50  0000 C CNN
-	1    4700 3150
-	-1   0    0    1
+P 7000 3050
+AR Path="/5881CF01" Ref="P6"  Part="1"
+AR Path="/5881B945/5881CF01" Ref="P6"  Part="1"
+F 0 "P6" H 7000 3200 50  0000 C CNN
+F 1 "Power_OUT" V 7100 3050 50  0000 C CNN
+F 2 "Terminal_Blocks:TerminalBlock_Pheonix_MKDS1.5-2pol" H 7000 3050 50  0001 C CNN
+F 3 "" H 7000 3050 50  0000 C CNN
+	1    7000 3050
+	1    0    0    -1
 $EndComp
 Text HLabel 7650 3550 2    60   Input ~ 0
@@
 ALERT
 $Comp
-L R_Small R13
+L Device:R_Small R13
 U 1 1 58841DD5
 P 7250 3100
@@
 $EndComp
 $Comp
-L R_Small R14
+L Device:R_Small R14
 U 1 1 58841E1B
 P 7400 3300
@@
 $EndComp
 $Comp
-L R_Small R15
+L Device:R_Small R15
 U 1 1 58841E6E
 P 7600 3400
@@
 $EndComp
 $Comp
-L C_Small C4
+L Device:C_Small C4
 U 1 1 58842FC4
 P 6850 4000
@@
 $EndComp
 $Comp
-L C_Small C5
+L Device:C_Small C5
 U 1 1 58847B1B
 P 5250 3550
@@
 $EndComp
 $Comp
-L +3.3VA #PWR014
+L power:+3.3VA #PWR014
 U 1 1 588F0CB3
 P 6950 3850
@@
 $EndComp
 $Comp
-L +3.3VA #PWR015
+L power:+3.3VA #PWR015
 U 1 1 588F18A1
 P 4700 3650
@@
 $EndComp
 $Comp
-L +3.3VA #PWR016
+L power:+3.3VA #PWR016
 U 1 1 588F1952
 P 4700 4150
@@
 $EndComp
 $Comp
-L +3.3VA #PWR017
+L power:+3.3VA #PWR017
 U 1 1 588F1A71
 P 7250 3000
@@
 $EndComp
 $Comp
-L GNDA #PWR018
+L power:GNDA #PWR018
 U 1 1 588F1B2E
 P 4700 4250
@@
 $EndComp
 $Comp
-L GNDA #PWR019
+L power:GNDA #PWR019
 U 1 1 588F1B73
 P 4700 3750
@@
 $EndComp
 $Comp
-L GNDA #PWR020
+L power:GNDA #PWR020
 U 1 1 588F1C0C
 P 5050 2850
@@
 $EndComp
 $Comp
-L GNDA #PWR021
+L power:GNDA #PWR021
 U 1 1 588F1CBD
 P 6700 2850
@@
 $EndComp
 $Comp
-L GNDA #PWR022
+L power:GNDA #PWR022
 U 1 1 588F1D56
 P 6700 4100
@@
 $EndComp
 $Comp
-L GNDA #PWR023
+L power:GNDA #PWR023
 U 1 1 588F1F34
 P 5250 3650
@@
 	4700 4250 4850 4250
 Wire Wire Line
-	5050 3650 5050 3800
-Wire Wire Line
-	5150 3950 5150 4250
+	5050 3650 5050 3750
+Wire Wire Line
+	5150 3950 5150 4150
 Wire Wire Line
 	6700 4000 6700 4100
@@
 	6700 4000 7150 4000
 Wire Wire Line
-	6700 3900 7150 3900
+	6700 3900 6850 3900
 Connection ~ 6950 3900
 Wire Wire Line
-	6700 3150 6700 3400
+	6700 3150 6700 3200
 Connection ~ 6700 3300
 Connection ~ 5350 3300
 Connection ~ 5350 3400
 Wire Wire Line
-	6700 3750 7750 3750
+	6700 3750 7600 3750
 Wire Wire Line
 	6950 3850 6950 3900
 Connection ~ 5350 3200
-Connection ~ 6700 3400
 Connection ~ 6700 3200
 Wire Wire Line
@@
 Connection ~ 7600 3750
 Wire Wire Line
-	6700 3650 7700 3650
-Wire Wire Line
-	6700 3550 7650 3550
+	6700 3650 7400 3650
+Wire Wire Line
+	6700 3550 7250 3550
 Wire Wire Line
 	7400 3400 7400 3650
@@
 Connection ~ 5150 4150
 Wire Wire Line
-	5350 3200 5350 3600
+	5350 3200 5350 3300
 Wire Wire Line
 	5350 3200 4900 3200
@@
 	7400 3000 7400 3200
 Connection ~ 7250 3000
+Wire Wire Line
+	6950 3900 7150 3900
+Wire Wire Line
+	6700 3300 6700 3400
+Wire Wire Line
+	5350 3300 5350 3400
+Wire Wire Line
+	5350 3400 5350 3450
+Wire Wire Line
+	6700 3200 6700 3300
+Wire Wire Line
+	7600 3750 7750 3750
+Wire Wire Line
+	7400 3650 7700 3650
+Wire Wire Line
+	7250 3550 7650 3550
+Wire Wire Line
+	6850 3900 6950 3900
+Wire Wire Line
+	5350 3450 5350 3600
+Wire Wire Line
+	5050 3750 5050 3800
+Wire Wire Line
+	5150 4150 5150 4250
+$Comp
+L Connector:Screw_Terminal_01x02 P5
+U 1 1 5881CF96
+P 4700 3200
+AR Path="/5881CF96" Ref="P5"  Part="1"
+AR Path="/5881B945/5881CF96" Ref="P5"  Part="1"
+F 0 "P5" H 4700 3350 50  0000 C CNN
+F 1 "Power_IN" V 4800 3200 50  0000 C CNN
+F 2 "Terminal_Blocks:TerminalBlock_Pheonix_MKDS1.5-2pol" H 4700 3200 50  0001 C CNN
+F 3 "" H 4700 3200 50  0000 C CNN
+	1    4700 3200
+	-1   0    0    1
+$EndComp
 $EndSCHEMATC
