File: schematics/draw.sch (KiCad schematic (older format))
At the start: 31 parts, among them J1 USB_B_Micro, J2 Debug Header, P1 Power, SW1 SW_Push, U1 INA260, U2 TPD4E002, U3 EFM32HG309

Commit message: changed resistors to 4K7
Parts:
- R3, R4, R5: value 1K -> 4K7
Changed lines of the file:
@@
 P 3100 5050
 F 0 "R3" H 3130 5070 50  0000 L CNN
-F 1 "1K" H 3130 5010 50  0000 L CNN
+F 1 "4K7" H 2900 5050 50  0000 L CNN
 F 2 "Resistors_SMD:R_0805_HandSoldering" H 3100 5050 50  0001 C CNN
 F 3 "" H 3100 5050 50  0000 C CNN
@@
 P 3250 5250
 F 0 "R4" H 3280 5270 50  0000 L CNN
-F 1 "1K" H 3280 5210 50  0000 L CNN
+F 1 "4K7" H 3280 5210 50  0000 L CNN
 F 2 "Resistors_SMD:R_0805_HandSoldering" H 3250 5250 50  0001 C CNN
 F 3 "" H 3250 5250 50  0000 C CNN
@@
 P 3450 5350
 F 0 "R5" H 3480 5370 50  0000 L CNN
-F 1 "1K" H 3480 5310 50  0000 L CNN
+F 1 "4K7" H 3480 5310 50  0000 L CNN
 F 2 "Resistors_SMD:R_0805_HandSoldering" H 3450 5350 50  0001 C CNN
 F 3 "" H 3450 5350 50  0000 C CNN

Commit message: added VBUS and GND Power headers
Parts:
- removed P1: Power, Terminal_Blocks:TerminalBlock_Pheonix_MKDS1.5-2pol, symbol Connector:Screw_Terminal_01x02
- added J1: Power, symbol Connector:Screw_Terminal_01x04
- renumbered J1 to J2, J2 to J3
Connections:
- net GND: now also J1.1 (Pin_1)
- net at JP1.1 (A), U1.1 (IN+), U1.2 (IN+)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: now also J1.3 (Pin_3)
- net at JP1.2 (B), U1.12 (VBUS): now also J1.2 (Pin_2)
- net at U1.14 (IN-), U1.15 (IN-), U1.16 (IN-): now also J1.4 (Pin_4)
Other:
- moved on the sheet: C1, JP1, R3, R4, R5, U1

Commit message: updating footprint assignment
Parts:
- removed J1: Power, symbol Connector:Screw_Terminal_01x04
- added J1: Conn_01x02_Female, Connector_PinHeader_1.00mm:PinHeader_1x02_P1.00mm_Vertical, symbol Connector:Conn_01x02_Female
- added J3: Screw_Terminal_01x02, TerminalBlock_MetzConnect:TerminalBlock_MetzConnect_Type086_RT03402HBLC_1x02_P3.81mm_Horizontal, symbol Connector:Screw_Terminal_01x02
- C1, C2, C3, C4, C5: footprint Capacitors_SMD:C_0805_HandSoldering -> Capacitor_SMD:C_0805_2012Metric_Pad1.15x1.40mm_HandSolder
- D1, D3: footprint LEDs:LED_0805 -> LED_SMD:LED_0805_2012Metric_Pad1.15x1.40mm_HandSolder
- D2: footprint (none) -> Diode_SMD:D_0805_2012Metric_Pad1.15x1.40mm_HandSolder
- J2: footprint (none) -> Connector_USB:USB_Micro-B_Amphenol_10103594-0001LF_Horizontal
- J4: renamed from J3; footprint (none) -> Connector_PinSocket_2.54mm:PinSocket_1x06_P2.54mm_Vertical
- JP1: footprint (none) -> Jumper:SolderJumper-2_P1.3mm_Open_RoundedPad1.0x1.5mm
- L1: footprint Capacitors_SMD:C_0805_HandSoldering -> Inductor_SMD:L_0805_2012Metric_Pad1.15x1.40mm_HandSolder
- R1, R2, R3, R4, R5, R6, R7: footprint Resistors_SMD:R_0805_HandSoldering -> Resistor_SMD:R_0805_2012Metric_Pad1.15x1.40mm_HandSolder
- TP1, TP2, TP3, TP4, TP5, TP6, TP7: footprint (none) -> TestPoint:TestPoint_Pad_2.0x2.0mm
- U1: footprint Housings_SSOP:TSSOP-16_4.4x5mm_Pitch0.65mm -> Package_SO:TSSOP-16_4.4x5mm_P0.65mm
- U2: footprint TO_SOT_Packages_SMD:SOT-553 -> Package_TO_SOT_SMD:SOT-553
- U3: footprint Housings_DFN_QFN:QFN-24-1EP_5x5mm_Pitch0.65mm -> Package_DFN_QFN:QFN-24-1EP_5x5mm_P0.65mm_EP3.6x3.6mm
Connections:
- net GND: now also J1.1 (Pin_1)
- net at JP1.1 (A), U1.1 (IN+), U1.2 (IN+)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: now also J3.1 (Pin_1)
- net at JP1.2 (B), U1.12 (VBUS): now also J1.2 (Pin_2)
- net at U1.14 (IN-), U1.15 (IN-), U1.16 (IN-): now also J3.2 (Pin_2)
Other:
- note added: "IN+\nIN-\n"
- note added: "VBUS\nGND\n"
